File: CAD/uplc-analog/uplc-analog.kicad_sch (KiCad schematic)
At the start: 49 parts, among them J1 Conn_01x06_Pin, J2 SM12B-GHS-TB(LF)(SN), U1 AP63201WU, U2 ADS1115IDGS, U3 ESP32-C3-WROOM-02, U4 LP5907MFX-3.0, U5 MCP4725xxx-xCH, Y1 32.768khz 3215 12.5pf

Commit message: Rev 1.1
Connections:
- net ADC_DRDY: now also U3.10 (GPIO10)
Changed lines of the file:
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@@
     (title "uPLC-Digital")
     (date "2024-02-22")
-    (rev "1.0.0")
+    (rev "1.1.0")
     (company "Drawn by FNB")
     (comment 1 "Thanks to https://github.com/PricelessToolkit/ESPClicker for inspiration")
@@
     )
   )
-  (global_label "ADC_DRDY" (shape input) (at 135.89 31.75 0) (fields_autoplaced)
-    (effects (font (size 1.27 1.27)) (justify left))
-    (property "Intersheetrefs" "${INTERSHEET_REFS}" (at 148.37 31.75 0)
-      (effects (font (size 1.27 1.27)) (justify left) hide)
-    )
+  (global_label "ADC_DRDY" (shape input) (at 120.65 71.12 0) (fields_autoplaced)
+    (effects (font (size 1.27 1.27)) (justify left))
+    (property "Intersheetrefs" "${INTERSHEET_REFS}" (at 133.13 71.12 0)
+      (effects (font (size 1.27 1.27)) (justify left) hide)
+    )

Commit message: Panelization changes
Parts:
- R7: LCSC Part # (none) -> C159040
- U2: LCSC Part # (none) -> C37593
- U4: LCSC Part # (none) -> C475492
- U5: LCSC Part # (none) -> C144198

Commit message: feat: Production update
Parts:
- C1, C4: Generic (none) -> x; MPN (none) -> 0402CG200J500NT
- C10, C13, C14, C15, C16, C17, C18, C2, C3, C6, C9: Generic (none) -> x; LCSC Part # C307331 -> C77020; MPN (none) -> GRM155R71H104KE14D
- C11, C12, C8: Generic (none) -> x; MPN (none) -> GRM155R60J226ME11D
- C19, C20: value 1uF -> 0.1uF; Generic (none) -> x; LCSC Part # C307331 -> C77020; MPN (none) -> GRM155R71H104KE14D
- C5, C7: Generic (none) -> x; MPN (none) -> GRM21BR6YA106KE43L
- D1, D2, D3, D4: MPN (none) -> 1N5819WS
- J2: MPN (none) -> SM12B-GHS-TB(LF)(SN)
- L1: value 6.8uH -> 4.7uH; Generic (none) -> x; LCSC Part # C98340 -> C82314; MPN (none) -> LQM2HPN4R7MG0L
- R1, R12, R16, R2, R3, R4, R5, R6: Generic (none) -> x; MPN (none) -> 0402WGF1002TCE
- R10, R11, R8, R9: Generic (none) -> x; LCSC Part # C25076 -> C4125; MPN (none) -> 0402WGF4990TCE
- R13: Generic (none) -> x; MPN (none) -> 0402WGF1000TCE
- R14: Generic (none) -> x; MPN (none) -> 0402WGF1823TCE
- R15: Generic (none) -> x; MPN (none) -> RC0402FR-0762KL
- R7: Generic (none) -> x; MPN (none) -> RTT023093FTH
- U1: MPN (none) -> AP63201WU-7
- U2: MPN (none) -> ADS1115IDGSR
- U3: MPN (none) -> ESP32-C3-WROOM-02-N4
- U4: MPN (none) -> LP5907MFX-3.0/NOPB
- U5: MPN (none) -> MCP4725A0T-E/CH
- Y1: MPN (none) -> Q13FC13500004
